File: ether_v1/ether_v1.kicad_pcb (KiCad board)
At the start: 2 copper layers, 214 x 79 mm, 39 parts, among them J1 AudioJack2_SwitchT, J10 AudioJack2_SwitchT, J11 AudioJack2_SwitchT, J12 AudioJack2_SwitchT, J13 AudioJack2_SwitchT, J14 AudioJack2_SwitchT, J15 AudioJack2_SwitchT, J16 AudioJack2_SwitchT, J17 1-406541-5, J18 1-406541-5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

Commit message: Add Ether Twin v1 README, bom, schematic.
Parts:
- renumbered mouse-bite-2mm-slot to MH
Other:
- board text added: "1A"
- board text added: "1B"
- board text added: "2A"
- board text added: "2B"
- board text added: "3A"
- board text added: "3B"
- board text added: "4A"
- board text added: "4B"
- board text added: "5A"
- board text added: "5B"
- board text added: "6A"
- board text added: "6B"
- board text added: "7A"
- board text added: "7B"
- board text added: "8A"
- board text added: "8B"
- board text added: "CAT6"
- board text added: "Ether Twin v1.2 2024-03-01 Designed by Adam Wonak & Dom Pinchott github.com/awonak/ether-twin"
- board text added: "GROUND"
- board text added: "JLCJLCJLCJLC"
- board text removed: "A1"
- board text removed: "A2"
- board text removed: "A3"
- board text removed: "A4"
- board text removed: "A5"
- board text removed: "A6"
- board text removed: "A7"
- board text removed: "A8"
- board text removed: "B1"
- board text removed: "B2"
- board text removed: "B3"
- board text removed: "B4"
- board text removed: "B5"
- board text removed: "B6"
- board text removed: "B7"
Changed lines of the file:
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@@
     (fp_circle (center 0 0.005) (end 1.8 0.005)
       (stroke (width 0.1) (type solid)) (fill none) (layer "F.Fab"))
-    (pad "S" thru_hole roundrect (at 0 -6.475) (size 1.93 1.83) (drill 1.5) (layers "*.Cu" "*.Mask") (roundrect_rratio 0.15)
+    (pad "S" thru_hole roundrect (at 0 -6.475) (size 1.93 2.2) (drill oval 1.5 1.8) (layers "*.Cu" "*.Mask") (roundrect_rratio 0.15)
       (net 1 "GND") (pintype "passive"))
     (pad "T" thru_hole circle (at 0 4.925) (size 2.13 2.13) (drill 1.43) (layers "*.Cu" "*.Mask")
@@
     (fp_circle (center 0 0.005) (end 1.8 0.005)
       (stroke (width 0.1) (type solid)) (fill none) (layer "F.Fab"))
-    (pad "S" thru_hole roundrect (at 0 -6.475) (size 1.93 1.83) (drill 1.5) (layers "*.Cu" "*.Mask") (roundrect_rratio 0.15)
+    (pad "S" thru_hole roundrect (at 0 -6.475) (size 1.93 2.2) (drill oval 1.5 1.8) (layers "*.Cu" "*.Mask") (roundrect_rratio 0.15)
       (net 1 "GND") (pintype "passive"))
     (pad "T" thru_hole circle (at 0 4.925) (size 2.13 2.13) (drill 1.43) (layers "*.Cu" "*.Mask")
@@
     (at 121 119 90)
     (attr through_hole)
-    (fp_text reference "mouse-bite-2mm-slot" (at 0 -2 90) (layer "F.SilkS") hide
+    (fp_text reference "MH" (at 0 -2 90) (layer "F.SilkS") hide
         (effects (font (size 1 1) (thickness 0.2)))
     )
@@
     (at 121 60.1 90)
     (attr through_hole)
-    (fp_text reference "mouse-bite-2mm-slot" (at 0 -2 90) (layer "F.SilkS") hide
+    (fp_text reference "MH" (at 0 -2 90) (layer "F.SilkS") hide
         (effects (font (size 1 1) (thickness 0.2)))
     )
@@
     (at 193 119 90)
     (attr through_hole)
-    (fp_text reference "mouse-bite-2mm-slot" (at 0 -2 90) (layer "F.SilkS") hide
+    (fp_text reference "MH" (at 0 -2 90) (layer "F.SilkS") hide
         (effects (font (size 1 1) (thickness 0.2)))
     )
@@
     (fp_circle (center 0 0.005) (end 1.8 0.005)
       (stroke (width 0.1) (type solid)) (fill none) (layer "F.Fab"))
-    (pad "S" thru_hole roundrect (at 0 -6.475) (size 1.93 1.83) (drill 1.5) (layers "*.Cu" "*.Mask") (roundrect_rratio 0.15)
+    (pad "S" thru_hole roundrect (at 0 -6.475) (size 1.93 2.2) (drill oval 1.5 1.8) (layers "*.Cu" "*.Mask") (roundrect_rratio 0.15)
       (net 1 "GND") (pintype "passive"))
     (pad "T" thru_hole circle (at 0 4.925) (size 2.13 2.13) (drill 1.43) (layers "*.Cu" "*.Mask")
@@
     (fp_circle (center 0 0.005) (end 1.8 0.005)
       (stroke (width 0.1) (type solid)) (fill none) (layer "F.Fab"))
-    (pad "S" thru_hole roundrect (at 0 -6.475) (size 1.93 1.83) (drill 1.5) (layers "*.Cu" "*.Mask") (roundrect_rratio 0.15)
+    (pad "S" thru_hole roundrect (at 0 -6.475) (size 1.93 2.2) (drill oval 1.5 1.8) (layers "*.Cu" "*.Mask") (roundrect_rratio 0.15)
       (net 1 "GND") (pintype "passive"))
     (pad "T" thru_hole circle (at 0 4.925) (size 2.13 2.13) (drill 1.43) (layers "*.Cu" "*.Mask")
@@
     (property "SnapEDA_Link" "https://www.snapeda.com/parts/JS102011SAQN/C%2526K/view-part/?ref=snap")
     (attr smd)
-    (fp_text reference "S5" (at -0.438995 -5.175125 90) (layer "F.SilkS")
+    (fp_text reference "S5" (at 5.171375 -1.134505 180) (layer "F.SilkS")
         (effects (font (size 1.000732 1.000732) (thickness 0.15)))
     )
@@
     (at 193 60.1 90)
     (attr through_hole)
-    (fp_text reference "mouse-bite-2mm-slot" (at 0 -2 90) (layer "F.SilkS") hide
+    (fp_text reference "MH" (at 0 -2 90) (layer "F.SilkS") hide
         (effects (font (size 1 1) (thickness 0.2)))
     )
@@
   (gr_circle (center 203 77.1) (end 206.05 77.1)
     (stroke (width 0.1) (type default)) (fill none) (layer "Edge.Cuts"))
-  (gr_text "B5" (at 245.9 106.4) (layer "F.SilkS")
+  (gr_text "JLCJLCJLCJLC" (at 157.1 126) (layer "B.SilkS")
+    (effects (font (size 1 1) (thickness 0.15)) (justify mirror))
+  )
+  (gr_text "5B" (at 245.9 106.4) (layer "F.SilkS")
     (effects (font (size 2 2) (thickness 0.3) bold) (justify left bottom))
   )
-  (gr_text "A2" (at 208.15 76.65) (layer "F.SilkS")
+  (gr_text "2A" (at 208.15 76.65) (layer "F.SilkS")
     (effects (font (size 2 2) (thickness 0.3) bold) (justify left bottom))
   )
-  (gr_text "B6" (at 258.9 106.4) (layer "F.SilkS")
+  (gr_text "6B" (at 258.9 106.4) (layer "F.SilkS")
     (effects (font (size 2 2) (thickness 0.3) bold) (justify left bottom))
   )
@@
     (effects (font (size 1 1) (thickness 0.15)))
   )
-  (gr_text "A8" (at 208.15 115.7) (layer "F.SilkS")
+  (gr_text "8A" (at 208.15 115.7) (layer "F.SilkS")
     (effects (font (size 2 2) (thickness 0.3) bold) (justify left bottom))
   )
-  (gr_text "A4" (at 208.15 89.7) (layer "F.SilkS")
+  (gr_text "4A" (at 208.15 89.7) (layer "F.SilkS")
     (effects (font (size 2 2) (thickness 0.3) bold) (justify left bottom))
   )
@@
     (effects (font (size 4 4) (thickness 0.3)) (justify bottom))
   )
-  (gr_text "B8" (at 258.9 119.4) (layer "F.SilkS")
+  (gr_text "8B" (at 258.9 119.4) (layer "F.SilkS")
     (effects (font (size 2 2) (thickness 0.3) bold) (justify left bottom))
   )
-  (gr_text "A7" (at 195.3 115.7) (layer "F.SilkS")
+  (gr_text "7A" (at 195.3 115.7) (layer "F.SilkS")
     (effects (font (size 2 2) (thickness 0.3) bold) (justify left bottom))
   )
-  (gr_text "A1" (at 195.3 76.65) (layer "F.SilkS")
+  (gr_text "1A" (at 195.3 76.65) (layer "F.SilkS")
     (effects (font (size 2 2) (thickness 0.3) bold) (justify left bottom))
   )
-  (gr_text "B3" (at 245.9 93.4) (layer "F.SilkS")
+  (gr_text "3B" (at 245.9 93.4) (layer "F.SilkS")
     (effects (font (size 2 2) (thickness 0.3) bold) (justify left bottom))
   )
-  (gr_text "B1" (at 245.9 80.35) (layer "F.SilkS")
+  (gr_text "1B" (at 245.9 80.35) (layer "F.SilkS")
     (effects (font (size 2 2) (thickness 0.3) bold) (justify left bottom))
   )
-  (gr_text "B2" (at 258.9 80.35) (layer "F.SilkS")
+  (gr_text "2B" (at 258.9 80.35) (layer "F.SilkS")
     (effects (font (size 2 2) (thickness 0.3) bold) (justify left bottom))
   )
-  (gr_text "A3" (at 195.3 89.7) (layer "F.SilkS")
+  (gr_text "GROUND" (at 182.8 62.8 90) (layer "F.SilkS")
+    (effects (font (size 1 1) (thickness 0.15)))
+  )
+  (gr_text "CAT6" (at 191.1 67.7 90) (layer "F.SilkS")
+    (effects (font (size 1 1) (thickness 0.15)))
+  )
+  (gr_text "3A" (at 195.3 89.7) (layer "F.SilkS")
     (effects (font (size 2 2) (thickness 0.3) bold) (justify left bottom))
   )
-  (gr_text "ETHER TWIN" (at 85 101) (layer "F.SilkS")
+  (gr_text "ETHER TWIN" (at 85 61) (layer "F.SilkS")
     (effects (font (size 4 4) (thickness 0.3)) (justify bottom))
   )
-  (gr_text "A5" (at 195.3 102.7) (layer "F.SilkS")
+  (gr_text "5A" (at 195.3 102.7) (layer "F.SilkS")
     (effects (font (size 2 2) (thickness 0.3) bold) (justify left bottom))
   )
-  (gr_text "A6" (at 208.15 102.7) (layer "F.SilkS")
+  (gr_text "6A" (at 208.15 102.7) (layer "F.SilkS")
     (effects (font (size 2 2) (thickness 0.3) bold) (justify left bottom))
   )
-  (gr_text "B7" (at 245.9 119.4) (layer "F.SilkS")
+  (gr_text "B8" (at 191 58.7 90) (layer "F.SilkS")
+    (effects (font (size 1 1) (thickness 0.15)))
+  )
+  (gr_text "7B" (at 245.9 119.4) (layer "F.SilkS")
     (effects (font (size 2 2) (thickness 0.3) bold) (justify left bottom))
   )
-  (gr_text "passive chainable patch link over ethernet" (at 85 102.5) (layer "F.SilkS")
-    (effects (font (size 1.1 1.1) (thickness 0.15)) (justify bottom))
-  )
-  (gr_text "B4" (at 258.9 93.4) (layer "F.SilkS")
+  (gr_text "passive chainable patch link over ethernet" (at 85 62.5) (layer "F.SilkS")
+    (effects (font (size 1.1 1.05) (thickness 0.15)) (justify bottom))
+  )
+  (gr_text "4B" (at 258.9 93.4) (layer "F.SilkS")
     (effects (font (size 2 2) (thickness 0.3) bold) (justify left bottom))
   )
@@
     (effects (font (size 1 1) (thickness 0.2) bold) (justify bottom))
   )
+  (gr_text "GROUND" (at 262.4 62.7 90) (layer "F.SilkS")
+    (effects (font (size 1 1) (thickness 0.15)))
+  )
   (gr_text "passive chainable patch link over ethernet" (at 229 128.5) (layer "F.SilkS")
     (effects (font (size 1.1 1.1) (thickness 0.15)) (justify bottom))
   )
-  (gr_text "Ether Twin v1.2 2024-02-24\nDesigned by Adam Wonak & Dom Pinchott\ngithub.com/awonak/ether-twin\n" (at 85 109) (layer "F.SilkS")
+  (gr_text "Ether Twin v1.2 2024-03-01\nDesigned by Adam Wonak & Dom Pinchott\ngithub.com/awonak/ether-twin\n" (at 85 69) (layer "F.SilkS")
     (effects (font (size 1 1) (thickness 0.2) bold) (justify bottom))
   )
