File: ether_v1/ether_v1.kicad_sch (KiCad schematic)
At the start: 23 parts, among them J1 1-406541-5, J10 AudioJack2_SwitchT, J11 AudioJack2_SwitchT, J12 AudioJack2_SwitchT, J13 AudioJack2_SwitchT, J14 AudioJack2_SwitchT, J15 AudioJack2_SwitchT, J16 AudioJack2_SwitchT, J17 AudioJack2_SwitchT, J18 AudioJack2_SwitchT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

Commit message: Add Ether Twin v1 README, bom, schematic.
Other:
- title: (none) -> Ether Twin - Standalone
Changed lines of the file:
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@@
 (kicad_sch (version 20230121) (generator eeschema)
   (paper "A4")
+  (title_block
+    (title "Ether Twin - Standalone")
+    (date "2024-03-02")
+    (rev "v1.2")
+  )
   (junction (at 200.66 82.55) (diameter 0) (color 0 0 0 0)
   )
@@
         )
       )
-      (project "ether_v1.2"
+      (project "ether_v1"
         (path "/9e5b6781-8bb4-4cae-9d81-f975d4ca6a91"
           (reference "J16") (unit 1)
@@
     (pin "6")
     (instances
-      (project "ether_v1.2"
+      (project "ether_v1"
         (path "/9e5b6781-8bb4-4cae-9d81-f975d4ca6a91"
           (reference "S4") (unit 2)
@@
         )
       )
-      (project "ether_v1.2"
+      (project "ether_v1"
         (path "/9e5b6781-8bb4-4cae-9d81-f975d4ca6a91"
           (reference "J15") (unit 1)
@@
     (pin "6")
     (instances
-      (project "ether_v1.2"
+      (project "ether_v1"
         (path "/9e5b6781-8bb4-4cae-9d81-f975d4ca6a91"
           (reference "S4") (unit 1)
@@
     (pin "6")
     (instances
-      (project "ether_v1.2"
+      (project "ether_v1"
         (path "/9e5b6781-8bb4-4cae-9d81-f975d4ca6a91"
           (reference "S2") (unit 2)
@@
     (pin "6")
     (instances
-      (project "ether_v1.2"
+      (project "ether_v1"
         (path "/9e5b6781-8bb4-4cae-9d81-f975d4ca6a91"
           (reference "S2") (unit 1)
@@
         )
       )
-      (project "ether_v1.2"
+      (project "ether_v1"
         (path "/9e5b6781-8bb4-4cae-9d81-f975d4ca6a91"
           (reference "#PWR012") (unit 1)
@@
         )
       )
-      (project "ether_v1.2"
+      (project "ether_v1"
         (path "/9e5b6781-8bb4-4cae-9d81-f975d4ca6a91"
           (reference "#PWR07") (unit 1)
@@
         )
       )
-      (project "ether_v1.2"
+      (project "ether_v1"
         (path "/9e5b6781-8bb4-4cae-9d81-f975d4ca6a91"
           (reference "#PWR017") (unit 1)
@@
         )
       )
-      (project "ether_v1.2"
+      (project "ether_v1"
         (path "/9e5b6781-8bb4-4cae-9d81-f975d4ca6a91"
           (reference "#PWR05") (unit 1)
@@
         )
       )
-      (project "ether_v1.2"
+      (project "ether_v1"
         (path "/9e5b6781-8bb4-4cae-9d81-f975d4ca6a91"
           (reference "J3") (unit 1)
@@
         )
       )
-      (project "ether_v1.2"
+      (project "ether_v1"
         (path "/9e5b6781-8bb4-4cae-9d81-f975d4ca6a91"
           (reference "#PWR020") (unit 1)
@@
         )
       )
-      (project "ether_v1.2"
+      (project "ether_v1"
         (path "/9e5b6781-8bb4-4cae-9d81-f975d4ca6a91"
           (reference "J12") (unit 1)
@@
         )
       )
-      (project "ether_v1.2"
+      (project "ether_v1"
         (path "/9e5b6781-8bb4-4cae-9d81-f975d4ca6a91"
           (reference "J13") (unit 1)
@@
         )
       )
-      (project "ether_v1.2"
+      (project "ether_v1"
         (path "/9e5b6781-8bb4-4cae-9d81-f975d4ca6a91"
           (reference "#PWR015") (unit 1)
@@
         )
       )
-      (project "ether_v1.2"
+      (project "ether_v1"
         (path "/9e5b6781-8bb4-4cae-9d81-f975d4ca6a91"
           (reference "#PWR02") (unit 1)
@@
         )
       )
-      (project "ether_v1.2"
+      (project "ether_v1"
         (path "/9e5b6781-8bb4-4cae-9d81-f975d4ca6a91"
           (reference "J5") (unit 1)
@@
         )
       )
-      (project "ether_v1.2"
+      (project "ether_v1"
         (path "/9e5b6781-8bb4-4cae-9d81-f975d4ca6a91"
           (reference "S5") (unit 1)
@@
         )
       )
-      (project "ether_v1.2"
+      (project "ether_v1"
         (path "/9e5b6781-8bb4-4cae-9d81-f975d4ca6a91"
           (reference "J4") (unit 1)
@@
         )
       )
-      (project "ether_v1.2"
+      (project "ether_v1"
         (path "/9e5b6781-8bb4-4cae-9d81-f975d4ca6a91"
           (reference "#PWR06") (unit 1)
@@
         )
       )
-      (project "ether_v1.2"
+      (project "ether_v1"
         (path "/9e5b6781-8bb4-4cae-9d81-f975d4ca6a91"
           (reference "J10") (unit 1)
@@
         )
       )
-      (project "ether_v1.2"
+      (project "ether_v1"
         (path "/9e5b6781-8bb4-4cae-9d81-f975d4ca6a91"
           (reference "#PWR04") (unit 1)
@@
         )
       )
-      (project "ether_v1.2"
+      (project "ether_v1"
         (path "/9e5b6781-8bb4-4cae-9d81-f975d4ca6a91"
           (reference "#PWR01") (unit 1)
@@
         )
       )
-      (project "ether_v1.2"
+      (project "ether_v1"
         (path "/9e5b6781-8bb4-4cae-9d81-f975d4ca6a91"
           (reference "#PWR021") (unit 1)
@@
         )
       )
-      (project "ether_v1.2"
+      (project "ether_v1"
         (path "/9e5b6781-8bb4-4cae-9d81-f975d4ca6a91"
           (reference "J8") (unit 1)
@@
     (pin "6")
     (instances
-      (project "ether_v1.2"
+      (project "ether_v1"
         (path "/9e5b6781-8bb4-4cae-9d81-f975d4ca6a91"
           (reference "S3") (unit 2)
@@
         )
       )
-      (project "ether_v1.2"
+      (project "ether_v1"
         (path "/9e5b6781-8bb4-4cae-9d81-f975d4ca6a91"
           (reference "#PWR09") (unit 1)
@@
         )
       )
-      (project "ether_v1.2"
+      (project "ether_v1"
         (path "/9e5b6781-8bb4-4cae-9d81-f975d4ca6a91"
           (reference "#PWR010") (unit 1)
@@
         )
       )
-      (project "ether_v1.2"
+      (project "ether_v1"
         (path "/9e5b6781-8bb4-4cae-9d81-f975d4ca6a91"
           (reference "#PWR03") (unit 1)
@@
         )
       )
-      (project "ether_v1.2"
+      (project "ether_v1"
         (path "/9e5b6781-8bb4-4cae-9d81-f975d4ca6a91"
           (reference "#PWR013") (unit 1)
@@
     (pin "6")
     (instances
-      (project "ether_v1.2"
+      (project "ether_v1"
         (path "/9e5b6781-8bb4-4cae-9d81-f975d4ca6a91"
           (reference "S1") (unit 2)
@@
         )
       )
-      (project "ether_v1.2"
+      (project "ether_v1"
         (path "/9e5b6781-8bb4-4cae-9d81-f975d4ca6a91"
           (reference "#PWR018") (unit 1)
@@
         )
       )
-      (project "ether_v1.2"
+      (project "ether_v1"
         (path "/9e5b6781-8bb4-4cae-9d81-f975d4ca6a91"
           (reference "#PWR016") (unit 1)
@@
         )
       )
-      (project "ether_v1.2"
+      (project "ether_v1"
         (path "/9e5b6781-8bb4-4cae-9d81-f975d4ca6a91"
           (reference "#PWR011") (unit 1)
@@
     (pin "6")
     (instances
-      (project "ether_v1.2"
+      (project "ether_v1"
         (path "/9e5b6781-8bb4-4cae-9d81-f975d4ca6a91"
           (reference "S1") (unit 1)
@@
         )
       )
-      (project "ether_v1.2"
+      (project "ether_v1"
         (path "/9e5b6781-8bb4-4cae-9d81-f975d4ca6a91"
           (reference "J18") (unit 1)
@@
         )
       )
-      (project "ether_v1.2"
+      (project "ether_v1"
         (path "/9e5b6781-8bb4-4cae-9d81-f975d4ca6a91"
           (reference "J7") (unit 1)
@@
         )
       )
-      (project "ether_v1.2"
+      (project "ether_v1"
         (path "/9e5b6781-8bb4-4cae-9d81-f975d4ca6a91"
           (reference "#PWR014") (unit 1)
@@
         )
       )
-      (project "ether_v1.2"
+      (project "ether_v1"
         (path "/9e5b6781-8bb4-4cae-9d81-f975d4ca6a91"
           (reference "J9") (unit 1)
@@
         )
       )
-      (project "ether_v1.2"
+      (project "ether_v1"
         (path "/9e5b6781-8bb4-4cae-9d81-f975d4ca6a91"
           (reference "J2") (unit 1)
@@
         )
       )
-      (project "ether_v1.2"
+      (project "ether_v1"
         (path "/9e5b6781-8bb4-4cae-9d81-f975d4ca6a91"
           (reference "J17") (unit 1)
@@
         )
       )
-      (project "ether_v1.2"
+      (project "ether_v1"
         (path "/9e5b6781-8bb4-4cae-9d81-f975d4ca6a91"
           (reference "J14") (unit 1)
@@
         )
       )
-      (project "ether_v1.2"
+      (project "ether_v1"
         (path "/9e5b6781-8bb4-4cae-9d81-f975d4ca6a91"
           (reference "#PWR08") (unit 1)
@@
         )
       )
-      (project "ether_v1.2"
+      (project "ether_v1"
         (path "/9e5b6781-8bb4-4cae-9d81-f975d4ca6a91"
           (reference "J6") (unit 1)
@@
     (pin "6")
     (instances
-      (project "ether_v1.2"
+      (project "ether_v1"
         (path "/9e5b6781-8bb4-4cae-9d81-f975d4ca6a91"
           (reference "S3") (unit 1)
@@
         )
       )
-      (project "ether_v1.2"
+      (project "ether_v1"
         (path "/9e5b6781-8bb4-4cae-9d81-f975d4ca6a91"
           (reference "#PWR019") (unit 1)
@@
         )
       )
-      (project "ether_v1.2"
+      (project "ether_v1"
         (path "/9e5b6781-8bb4-4cae-9d81-f975d4ca6a91"
           (reference "J1") (unit 1)
@@
         )
       )
-      (project "ether_v1.2"
+      (project "ether_v1"
         (path "/9e5b6781-8bb4-4cae-9d81-f975d4ca6a91"
           (reference "J11") (unit 1)
