File: ether_v2/ether_panel.kicad_pcb (KiCad board)
At the start: 2 copper layers, 50.5 x 128.5 mm, 0 parts

Commit message: Add Ether Twin v1 README, bom, schematic.
Other:
- board text added: "1A"
- board text added: "1B"
- board text added: "2A"
- board text added: "2B"
- board text added: "3A"
- board text added: "3B"
- board text added: "4A"
- board text added: "4B"
- board text added: "5A"
- board text added: "5B"
- board text added: "6A"
- board text added: "6B"
- board text added: "7A"
- board text added: "7B"
- board text added: "8A"
- board text added: "8B"
- board text removed: "A1"
- board text removed: "A2"
- board text removed: "A3"
- board text removed: "A4"
- board text removed: "A5"
- board text removed: "A6"
- board text removed: "A7"
- board text removed: "A8"
- board text removed: "B1"
- board text removed: "B2"
- board text removed: "B3"
- board text removed: "B4"
- board text removed: "B5"
- board text removed: "B6"
- board text removed: "B7"
- board text removed: "B8"
