File: ether_v2/ether_v2.kicad_pcb (KiCad board)
At the start: 2 copper layers, 50.3 x 110 mm, 82 parts, among them J1 CV A1, J10 CV A6, J11 CV B5, J12 CV B6, J13 CV A7, J14 CV A8, J15 CV B7, J16 CV B8, J17 Ethernet A, J18 Ethernet B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

Commit message: Add Ether Twin v1 README, bom, schematic.
Parts:
- J1: value CV A1 -> PJ398SM
- J10: value CV A6 -> PJ398SM
- J11: value CV B5 -> PJ398SM
- J12: value CV B6 -> PJ398SM
- J13: value CV A7 -> PJ398SM
- J14: value CV A8 -> PJ398SM
- J15: value CV B7 -> PJ398SM
- J16: value CV B8 -> PJ398SM
- J17: value Ethernet A -> SS65100-024F
- J18: value Ethernet B -> SS65100-024F
- J2: value CV A2 -> PJ398SM
- J3: value CV B1 -> PJ398SM
- J4: value CV B2 -> PJ398SM
- J5: value CV A3 -> PJ398SM
- J6: value CV A4 -> PJ398SM
- J7: value CV B3 -> PJ398SM
- J8: value CV B4 -> PJ398SM
- J9: value CV A5 -> PJ398SM
Other:
- board text added: "Ether Twin v2.2 2024-03-01"
- board text added: "GROUND"
- board text removed: "Ether Twin v2.2 2024-02-23"
- board text removed: "ground"

Commit message: Fix incorrect placement of ground and led resistor. Fixes Odd wiring of LED in schematic. #1
Parts:
- moved R13 16.5 mm to (32.5, 92.2), turned to -90 degrees
- moved R25 16.5 mm to (32.5, 113.2), turned to -90 degrees
- moved R9 16.5 mm to (32.5, 71.2), turned to 90 degrees
- moved R29 1.33 mm to (48.9, 134.4), turned to 180 degrees
- moved R26 0.50 mm to (69.5, 106.0), turned to 180 degrees
- moved R30 0.50 mm to (69.0, 127.5)
- moved R31 0.50 mm to (41.0, 127.5), turned to 180 degrees
- moved R14 0.15 mm to (69.4, 85.4), turned to 180 degrees
- moved R10 0.13 mm to (69.4, 64.5), turned to 180 degrees
- turned R11 to 180 degrees
- turned R15 to 180 degrees
- turned R27 to 180 degrees
Connections:
- R10 pad 1: Net-(D3-A) -> GND
- R10 pad 2: GND -> Net-(D3-K)
- R11 pad 1: GND -> Net-(D2-K)
- R11 pad 2: Net-(D2-A) -> GND
- R12 pad 1: Net-(D4-A) -> GND
- R12 pad 2: GND -> Net-(D4-K)
- R13 pad 1: GND -> Net-(D5-K)
- R13 pad 2: Net-(D5-A) -> GND
- R14 pad 1: Net-(D7-A) -> GND
- R14 pad 2: GND -> Net-(D7-K)
- R15 pad 1: GND -> Net-(D6-K)
- R15 pad 2: Net-(D6-A) -> GND
- R16 pad 1: Net-(D8-A) -> GND
- R16 pad 2: GND -> Net-(D8-K)
- R25 pad 1: GND -> Net-(D9-K)
- R25 pad 2: Net-(D9-A) -> GND
- R26 pad 1: Net-(D11-A) -> GND
- R26 pad 2: GND -> Net-(D11-K)
- R27 pad 1: GND -> Net-(D10-K)
- R27 pad 2: Net-(D10-A) -> GND
- R28 pad 1: Net-(D12-A) -> GND
- R28 pad 2: GND -> Net-(D12-K)
- R29 pad 1: GND -> Net-(D13-K)
- R29 pad 2: Net-(D13-A) -> GND
- R30 pad 1: Net-(D15-A) -> GND
- R30 pad 2: GND -> Net-(D15-K)
- R31 pad 1: GND -> Net-(D14-K)
- R31 pad 2: Net-(D14-A) -> GND
- R32 pad 1: Net-(D16-A) -> GND
- R32 pad 2: GND -> Net-(D16-K)
- R9 pad 2: Net-(D1-A) -> Net-(D1-K)
Routing:
- net Net-(D11-K): track 6.81 -> 14.8 mm
- net Net-(D15-K): track 6.81 -> 14.8 mm
- net Net-(D7-K): track 6.81 -> 14.4 mm
- net Net-(D3-K): track 6.81 -> 14.3 mm
- net Net-(D14-A): track 13.1 -> 7.30 mm
- net Net-(D8-K): track 17.8 -> 23.6 mm
- net Net-(D4-K): track 17.8 -> 23.6 mm
- net Net-(D16-K): track 17.8 -> 23.6 mm
- net Net-(D12-K): track 17.8 -> 23.6 mm
- net Net-(D6-A): track 12.8 -> 7.30 mm
- net Net-(D2-A): track 12.8 -> 7.30 mm
- net Net-(D10-A): track 12.8 -> 7.30 mm
- net Net-(D9-K): track 20.3 -> 24.9 mm
- net Net-(D5-K): track 20.3 -> 24.9 mm
- net Net-(D1-K): track 20.3 -> 24.9 mm
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
Commit message: Update pcb revision silkscreen.
Other:
- board text added: "Ether Twin v2.3 2024-03-17"
- board text removed: "Ether Twin v2.2 2024-03-01"
Changed lines of the file:
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@@
   (gr_arc (start 79.4025 29.9975) (mid 80.109607 30.290393) (end 80.4025 30.9975)
     (stroke (width 0.1) (type default)) (layer "Edge.Cuts"))
-  (gr_text "Ether Twin\nv2.2 2024-03-01" (at 55.6025 32.7475) (layer "B.SilkS")
+  (gr_text "Ether Twin\nv2.3 2024-03-17" (at 55.6025 32.7475) (layer "B.SilkS")
     (effects (font (size 1 1) (thickness 0.15)) (justify mirror))
   )

Commit message: fix bad merge
Parts:
- moved R13 16.5 mm to (49.0, 92.5), turned to 0 degrees
- moved R25 16.5 mm to (49.0, 113.5), turned to 0 degrees
- moved R9 16.5 mm to (49.0, 71.5), turned to 0 degrees
- moved R29 1.33 mm to (49.9, 135.2), turned to 90 degrees
- moved R26 0.50 mm to (69.5, 106.5), turned to 0 degrees
- moved R30 0.50 mm to (69.5, 127.5)
- moved R31 0.50 mm to (41.0, 128.0), turned to 0 degrees
- moved R14 0.15 mm to (69.5, 85.5), turned to 0 degrees
- moved R10 0.13 mm to (69.5, 64.5), turned to 0 degrees
- turned R11 to 0 degrees
- turned R15 to 0 degrees
- turned R27 to 0 degrees
Connections:
- R10 pad 1: GND -> Net-(D3-A)
- R10 pad 2: Net-(D3-K) -> GND
- R11 pad 1: Net-(D2-K) -> GND
- R11 pad 2: GND -> Net-(D2-A)
- R12 pad 1: GND -> Net-(D4-A)
- R12 pad 2: Net-(D4-K) -> GND
- R13 pad 1: Net-(D5-K) -> GND
- R13 pad 2: GND -> Net-(D5-A)
- R14 pad 1: GND -> Net-(D7-A)
- R14 pad 2: Net-(D7-K) -> GND
- R15 pad 1: Net-(D6-K) -> GND
- R15 pad 2: GND -> Net-(D6-A)
- R16 pad 1: GND -> Net-(D8-A)
- R16 pad 2: Net-(D8-K) -> GND
- R25 pad 1: Net-(D9-K) -> GND
- R25 pad 2: GND -> Net-(D9-A)
- R26 pad 1: GND -> Net-(D11-A)
- R26 pad 2: Net-(D11-K) -> GND
- R27 pad 1: Net-(D10-K) -> GND
- R27 pad 2: GND -> Net-(D10-A)
- R28 pad 1: GND -> Net-(D12-A)
- R28 pad 2: Net-(D12-K) -> GND
- R29 pad 1: Net-(D13-K) -> GND
- R29 pad 2: GND -> Net-(D13-A)
- R30 pad 1: GND -> Net-(D15-A)
- R30 pad 2: Net-(D15-K) -> GND
- R31 pad 1: Net-(D14-K) -> GND
- R31 pad 2: GND -> Net-(D14-A)
- R32 pad 1: GND -> Net-(D16-A)
- R32 pad 2: Net-(D16-K) -> GND
- R9 pad 2: Net-(D1-K) -> Net-(D1-A)
Routing:
- net Net-(D11-K): track 14.8 -> 6.81 mm
- net Net-(D15-K): track 14.8 -> 6.81 mm
- net Net-(D7-K): track 14.4 -> 6.81 mm
- net Net-(D3-K): track 14.3 -> 6.81 mm
- net Net-(D14-A): track 7.30 -> 13.1 mm
- net Net-(D8-K): track 23.6 -> 17.8 mm
- net Net-(D4-K): track 23.6 -> 17.8 mm
- net Net-(D16-K): track 23.6 -> 17.8 mm
- net Net-(D12-K): track 23.6 -> 17.8 mm
- net Net-(D6-A): track 7.30 -> 12.8 mm
- net Net-(D2-A): track 7.30 -> 12.8 mm
- net Net-(D10-A): track 7.30 -> 12.8 mm
- net Net-(D9-K): track 24.9 -> 20.3 mm
- net Net-(D5-K): track 24.9 -> 20.3 mm
- net Net-(D1-K): track 24.9 -> 20.3 mm
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Other:
- board text added: "Ether Twin v2.2 2024-03-01"
- board text removed: "Ether Twin v2.3 2024-03-17"
